Commit message: loading change

File: resources/robots/a1/urdf/a1.urdf (robot description, URDF)
Before this commit: robot a1_description, 23 links, 22 joints
Links:
- added link back_box, mass 0.5; collision box size=0.01 0.22 0.15; collision box size=0.01 0.22 0.15
Joints:
- added joint trunk_to_back_box: type fixed, parent trunk, child back_box, origin xyz=0.00 0.0 0.114 rpy=0 0 0
